File: KiCad/RFM95/RFM95.kicad_pcb (KiCad board)
At the start: 2 copper layers, 1 part, among them U1 RFM95W-868S2

Commit message: Changes to the board
Parts:
- added J1: Conn_Coaxial, Connector_Coaxial:SMA_Amphenol_132134-16_Vertical, F.Cu at (152.4, 96.5)
Routing:
- net unconnected-(U1-SCK-Pad4): vias 0 -> 1
- net unconnected-(U1-NSS-Pad5): vias 0 -> 1
- net unconnected-(U1-MOSI-Pad3): vias 0 -> 1
- net unconnected-(U1-MISO-Pad2): vias 0 -> 1
- net Earth: vias 0 -> 1
- net (no net): vias 0 -> 11
Changed lines of the file:
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@@
   (net 13 "unconnected-(U1-DIO1-Pad15)")
   (net 14 "unconnected-(U1-DIO2-Pad16)")
+  (footprint "Connector_Coaxial:SMA_Amphenol_132134-16_Vertical" (layer "F.Cu")
+    (at 152.4 96.52)
+    (descr "https://www.amphenolrf.com/downloads/dl/file/id/1141/product/2978/132134_16_customer_drawing.pdf")
+    (tags "SMA THT Female Jack Vertical ExtendedLegs")
+    (property "Sheetfile" "RFM95.kicad_sch")
+    (property "Sheetname" "")
+    (property "ki_description" "coaxial connector (BNC, SMA, SMB, SMC, Cinch/RCA, LEMO, ...)")
+    (property "ki_keywords" "BNC SMA SMB SMC LEMO coaxial connector CINCH RCA")
+    (attr through_hole)
+    (fp_text reference "J1" (at 0 -4.75) (layer "F.SilkS")
+        (effects (font (size 1 1) (thickness 0.15)))
+    )
+    (fp_text value "Conn_Coaxial" (at 0 5) (layer "F.Fab")
+        (effects (font (size 1 1) (thickness 0.15)))
+    )
+    (fp_text user "${REFERENCE}" (at 0 0) (layer "F.Fab")
+        (effects (font (size 1 1) (thickness 0.15)))
+    )
+    (fp_line (start -3.68 -1.8) (end -3.68 1.8)
+      (stroke (width 0.12) (type solid)) (layer "F.SilkS"))
+    (fp_line (start -1.8 -3.68) (end 1.8 -3.68)
+      (stroke (width 0.12) (type solid)) (layer "F.SilkS"))
+    (fp_line (start -1.8 3.68) (end 1.8 3.68)
+      (stroke (width 0.12) (type solid)) (layer "F.SilkS"))
+    (fp_line (start 3.68 -1.8) (end 3.68 1.8)
+      (stroke (width 0.12) (type solid)) (layer "F.SilkS"))
+    (fp_line (start -4.17 -4.17) (end -4.17 4.17)
+      (stroke (width 0.05) (type solid)) (layer "F.CrtYd"))
+    (fp_line (start -4.17 -4.17) (end 4.17 -4.17)
+      (stroke (width 0.05) (type solid)) (layer "F.CrtYd"))
+    (fp_line (start 4.17 4.17) (end -4.17 4.17)
+      (stroke (width 0.05) (type solid)) (layer "F.CrtYd"))
+    (fp_line (start 4.17 4.17) (end 4.17 -4.17)
+      (stroke (width 0.05) (type solid)) (layer "F.CrtYd"))
+    (fp_line (start -3.5 -3.5) (end -3.5 3.5)
+      (stroke (width 0.1) (type solid)) (layer "F.Fab"))
+    (fp_line (start -3.5 -3.5) (end 3.5 -3.5)
+      (stroke (width 0.1) (type solid)) (layer "F.Fab"))
+    (fp_line (start -3.5 3.5) (end 3.5 3.5)
+      (stroke (width 0.1) (type solid)) (layer "F.Fab"))
+    (fp_line (start 3.5 -3.5) (end 3.5 3.5)
+      (stroke (width 0.1) (type solid)) (layer "F.Fab"))
+    (fp_circle (center 0 0) (end 3.175 0)
+      (stroke (width 0.1) (type solid)) (fill none) (layer "F.Fab"))
+    (pad "1" thru_hole circle (at 0 0) (size 2.05 2.05) (drill 1.5) (layers "*.Cu" "*.Mask")
+      (net 8 "Net-(J1-In)") (pinfunction "In") (pintype "passive"))
+    (pad "2" thru_hole circle (at -2.54 -2.54) (size 2.25 2.25) (drill 1.7) (layers "*.Cu" "*.Mask")
+      (net 1 "Earth") (pinfunction "Ext") (pintype "passive"))
+    (pad "2" thru_hole circle (at -2.54 2.54) (size 2.25 2.25) (drill 1.7) (layers "*.Cu" "*.Mask")
+      (net 1 "Earth") (pinfunction "Ext") (pintype "passive"))
+    (pad "2" thru_hole circle (at 2.54 -2.54) (size 2.25 2.25) (drill 1.7) (layers "*.Cu" "*.Mask")
+      (net 1 "Earth") (pinfunction "Ext") (pintype "passive"))
+    (pad "2" thru_hole circle (at 2.54 2.54) (size 2.25 2.25) (drill 1.7) (layers "*.Cu" "*.Mask")
+      (net 1 "Earth") (pinfunction "Ext") (pintype "passive"))
+    (model "${KICAD6_3DMODEL_DIR}/Connector_Coaxial.3dshapes/SMA_Amphenol_132134-16_Vertical.wrl"
+      (offset (xyz 0 0 0))
+      (scale (xyz 1 1 1))
+      (rotate (xyz 0 0 0))
+    )
+  )
   (footprint "Library:RFM95" (layer "F.Cu")
     (at 146.94 81.9)
@@
     (fp_rect (start 3.5 -7.75) (end 5.75 -5)
       (stroke (width 0.1) (type default)) (fill none) (layer "F.SilkS"))
+    (fp_rect (start -14.224 -8.636) (end 13.716 9.652)
+      (stroke (width 0.05) (type default)) (fill none) (layer "F.CrtYd"))
     (pad "1" connect oval (at -8 -7) (size 4 1.524) (layers "F.Cu" "F.Mask")
       (net 1 "Earth") (pinfunction "GND") (pintype "power_in"))
@@
       (net 14 "unconnected-(U1-DIO2-Pad16)") (pinfunction "DIO2") (pintype "bidirectional"))
   )
+  (via (at 129.54 88.9) (size 0.8) (drill 0.4) (layers "F.Cu" "B.Cu") (net 0))
+  (via (at 162.56 88.9) (size 0.8) (drill 0.4) (layers "F.Cu" "B.Cu") (net 0))
+  (via (at 129.54 86.36) (size 0.8) (drill 0.4) (layers "F.Cu" "B.Cu") (net 0))
+  (via (at 162.56 76.2) (size 0.8) (drill 0.4) (layers "F.Cu" "B.Cu") (net 0))
+  (via (at 162.56 78.74) (size 0.8) (drill 0.4) (layers "F.Cu" "B.Cu") (net 0))
+  (via (at 129.54 91.44) (size 0.8) (drill 0.4) (layers "F.Cu" "B.Cu") (net 0))
+  (via (at 162.56 73.66) (size 0.8) (drill 0.4) (layers "F.Cu" "B.Cu") (net 0))
+  (via (at 162.56 81.28) (size 0.8) (drill 0.4) (layers "F.Cu" "B.Cu") (net 0))
+  (via (at 162.56 83.82) (size 0.8) (drill 0.4) (layers "F.Cu" "B.Cu") (net 0))
+  (via (at 162.56 86.36) (size 0.8) (drill 0.4) (layers "F.Cu" "B.Cu") (net 0))
+  (via (at 162.56 91.44) (size 0.8) (drill 0.4) (layers "F.Cu" "B.Cu") (net 0))
+  (via (at 129.54 73.66) (size 0.8) (drill 0.4) (layers "F.Cu" "B.Cu") (free) (net 1))
+  (via (at 129.54 76.2) (size 0.8) (drill 0.4) (layers "F.Cu" "B.Cu") (free) (net 2))
+  (via (at 129.54 78.74) (size 0.8) (drill 0.4) (layers "F.Cu" "B.Cu") (free) (net 3))
+  (via (at 129.54 81.28) (size 0.8) (drill 0.4) (layers "F.Cu" "B.Cu") (free) (net 4))
+  (via (at 129.54 83.82) (size 0.8) (drill 0.4) (layers "F.Cu" "B.Cu") (free) (net 5))
 )
